File: pcb/kicad/_saved_robofriend.sch (KiCad schematic (older format))
At the start: 139 parts, among them J1 I2C, J10 BAT2, J11 5VIN, J12 BAT3, J13 3V3OUT, J14 3V3OUT, J15 SPI, J16 MON/AMP, J17 M1, J18 M2, J19 US4, J2 ADC1, J20 5VOUT, J21 5VOUT, J22 US3, J23 US2, J24 US1, J25 I2C, J26 I2C, J27 I2C, J28 ADC4, J3 ADC2, J30 PWR, J31 MLe, J32 USB_A_4_PIN, J33 GS2, J4 UART, J5 ADC3, J6 ADC4, J7 BAT1, J8 MRi, J9 12VOUT, K2 SCHRACK-RTx3, Q2 NMOS, Q3 NPN, Q4 PMOS, Q5 NMOS, Q6 NMOS, Q7 NMOS, Q8 NMOS, U1 Teensy++2.0, U2 LM4040, U3 INA193, U4 MCP6001, U5 LM3940-3.3, U6 TL331

Commit message: completed CvPcb to assosiate components and footprints
Parts:
- added C28: 470u, Capacitors_SMD:CP_Elec_8x10, symbol CP
- C11: renamed from C19; footprint Capacitors_SMD:CP_Elec_6.3x5.3 -> Capacitors_SMD:CP_Elec_6.3x5.8; Part No (none) -> EEEFK1C470P
- C12: renamed from C20; footprint Capacitors_SMD:CP_Elec_10x10 -> Capacitors_SMD:CP_Elec_8x10; Part No (none) -> EEEFK1C471P
- C4: renamed from C14; footprint Capacitors_SMD:CP_Elec_4x5.8 -> Capacitors_SMD:CP_Elec_4x5.7; Part No (none) -> EEE0JA330WR
- C5: renamed from C11; value 0.1u -> 100u; footprint (none) -> Capacitors_SMD:CP_Elec_6.3x5.7; Part No (none) -> EEE1CA101WAP
- C6: renamed from C27; footprint (none) -> Capacitors_SMD:CP_Elec_5x5.7; Part No (none) -> EEE1CA330WR
- R22: renamed from R16; Part No (none) -> ERJ-M1WSJ10MU
- RV2: Part No (none) -> 3296Y-1-104LF
- gave numbers to parts that had none: 3
- renumbered C13 to C1, C18 to C10, C21 to C13, C22 to C14, C3 to C15, C4 to C16, C12 to C17, C23 to C18, C24 to C19, C1 to C2, C5 to C20, C25 to C21, C6 to C22, C9 to C23, C26 to C24, C10 to C25, C7 to C26, C8 to C27, C2 to C3, C15 to C7, C16 to C8, C17 to C9, D10 to D1, D19 to D10, D8 to D11, D9 to D12, D20 to D13, D21 to D14, D12 to D15, D23 to D16, D13 to D17, D2 to D18, D3 to D19, D24 to D2, D22 to D20, D6 to D21, D7 to D22, D4 to D23, D5 to D24, D11 to D3, D1 to D4, D14 to D5, D15 to D6, D16 to D7, D17 to D8, D18 to D9, J7 to J1, J22 to J10, J19 to J11, J1 to J12, J25 to J13, J26 to J14, J27 to J15, J9 to J16, J11 to J17, J20 to J18, J21 to J19, J10 to J2, J32 to J20, J16 to J21, J6 to J22, J8 to J23, J15 to J24, J28 to J25, J31 to J26, J17 to J27, J18 to J28, J2 to J29, J12 to J3, J3 to J30, J4 to J31, J5 to J32, J30 to J4, J24 to J5, J13 to J6, J14 to J7, J23 to J9, JP6 to JP2, JP7 to JP3, JP3 to JP4, JP4 to JP5, JP2 to JP6, JP5 to JP7, K2 to K1, Q2 to Q1, Q7 to Q2, Q8 to Q3, Q3 to Q4, Q4 to Q5, Q5 to Q6, Q6 to Q7, R9 to R1, R26 to R10, R27 to R11, R5 to R12, R31 to R13, R10 to R14, R12 to R15, R11 to R16, R13 to R17, R32 to R18, R21 to R19, R19 to R2, R14 to R20, R15 to R21, R2 to R23, R17 to R24, R18 to R25, R4 to R26, R22 to R27, R23 to R28, R3 to R29, R20 to R3, R24 to R30, R25 to R31, R28 to R4, R1 to R6, R6 to R7, R7 to R8, R8 to R9, U5 to U1, U1 to U2, U2 to U4, U4 to U5, U3 to U6, U6 to U7
